File: hardware/u2f-zero.sch (KiCad schematic (older format))
At the start: 10 parts, among them SW1 SW_PUSH

Commit message: updated schematic/pcb for pca pins, debug header, and udfn8
Parts:
- added DBG1: debug-header, footprints:debug, symbol debug-header
- A1: footprint SMD_Packages:SOIC-8-N -> footprints:UDFN-8Pad
Connections:
- net labels added: C2CK, C2D
- wire segments 39 -> 45
- no-connect marks 12 -> 8
Other:
- moved on the sheet: R1, RGB1, SW1
Changed lines of the file:
@@
 LIBS:atmel_cryptoauth
 LIBS:discrete
+LIBS:debug
 LIBS:u2f-zero-cache
 EELAYER 25 0
@@
 F 0 "A1" H 7300 5000 60  0000 C CNN
 F 1 "ATECC508A" H 6900 5000 60  0000 C CNN
-F 2 "SMD_Packages:SOIC-8-N" H 6600 4950 60  0001 C CNN
+F 2 "footprints:UDFN-8Pad" H 6600 4950 60  0001 C CNN
 F 3 "" H 6600 4950 60  0000 C CNN
 	1    7000 4700
@@
 NoConn ~ 7600 4850
 NoConn ~ 6400 4750
-NoConn ~ 6050 4400
-NoConn ~ 6050 4250
 Text Label 7850 5050 0    60   ~ 0
 GND
@@
 Text Label 4750 5450 2    60   ~ 0
 +3.3V
-Text Label 7350 3600 0    60   ~ 0
+Text Label 5450 2700 0    60   ~ 0
 +5V
-NoConn ~ 4350 4150
-NoConn ~ 4350 4300
 $Comp
 L DF5A5.6JE Z1
@@
 Text Label 3950 4750 2    60   ~ 0
 HD+
-Text Label 4350 3400 2    60   ~ 0
+Text Label 7100 3900 0    60   ~ 0
 GND
 $Comp
 L R R1
 U 1 1 56857B9B
-P 7050 3450
-F 0 "R1" V 7130 3450 50  0000 C CNN
-F 1 "100" V 7050 3450 50  0000 C CNN
-F 2 "Resistors_SMD:R_0603" V 6980 3450 50  0001 C CNN
-F 3 "" H 7050 3450 50  0000 C CNN
-	1    7050 3450
+P 5100 2700
+F 0 "R1" V 5180 2700 50  0000 C CNN
+F 1 "100" V 5100 2700 50  0000 C CNN
+F 2 "Resistors_SMD:R_0603" V 5030 2700 50  0001 C CNN
+F 3 "" H 5100 2700 50  0000 C CNN
+	1    5100 2700
 	0    1    1    0
 $EndComp
 NoConn ~ 5050 5300
-NoConn ~ 5200 5300
-NoConn ~ 5350 5300
 Text Notes 3050 3750 0    60   ~ 0
 Protect from ESD
@@
 L CA_RGB-RESCUE-u2f-zero RGB1
 U 1 1 5686DEFD
-P 6250 3650
-F 0 "RGB1" H 6500 3800 60  0000 C CNN
-F 1 "CA_RGB" H 6150 3800 60  0000 C CNN
-F 2 "footprints:LED-0606" H 7050 3700 60  0001 C CNN
-F 3 "" H 6250 3700 60  0000 C CNN
-	1    6250 3650
-	1    0    0    1
+P 4500 3200
+F 0 "RGB1" H 4750 3350 60  0000 C CNN
+F 1 "CA_RGB" H 4400 3350 60  0000 C CNN
+F 2 "footprints:LED-0606" H 5300 3250 60  0001 C CNN
+F 3 "" H 4500 3250 60  0000 C CNN
+	1    4500 3200
+	0    1    -1   0
 $EndComp
 $Comp
@@
 	7850 4550 7850 5050
 Wire Wire Line
-	7200 3450 7350 3450
-Wire Wire Line
-	7350 3450 7350 3600
-Wire Wire Line
 	4900 5300 4900 6150
 Wire Wire Line
@@
 Wire Wire Line
 	5500 5600 5900 5600
-Wire Wire Line
-	5100 3400 5100 3700
-Wire Wire Line
-	4500 3400 4350 3400
-Wire Wire Line
-	6900 3450 6750 3450
-Wire Wire Line
-	5550 3700 5550 3600
-Wire Wire Line
-	5550 3600 5800 3600
-Wire Wire Line
-	5800 3450 5400 3450
-Wire Wire Line
-	5400 3450 5400 3700
-Wire Wire Line
-	5250 3700 5250 3300
-Wire Wire Line
-	5250 3300 5800 3300
 Wire Wire Line
 	6850 5850 6850 5650
@@
 L SW_PUSH SW1
 U 1 1 5685E9F9
-P 4800 3400
-F 0 "SW1" H 4950 3510 50  0000 C CNN
-F 1 "SW_PUSH" H 4800 3320 50  0000 C CNN
-F 2 "footprints:MJTP1230" H 4800 3400 50  0001 C CNN
-F 3 "" H 4800 3400 50  0000 C CNN
-	1    4800 3400
+P 6650 3900
+F 0 "SW1" H 6800 4010 50  0000 C CNN
+F 1 "SW_PUSH" H 6650 3820 50  0000 C CNN
+F 2 "footprints:MJTP1230" H 6650 3900 50  0001 C CNN
+F 3 "" H 6650 3900 50  0000 C CNN
+	1    6650 3900
 	1    0    0    -1
 $EndComp
-Wire Wire Line
-	4950 3700 4950 3650
-Wire Wire Line
-	4950 3650 5100 3650
-Connection ~ 5100 3650
 Wire Wire Line
 	3300 4600 3300 4750
@@
 Wire Wire Line
 	3650 4000 3650 3900
+Wire Wire Line
+	6050 4250 6050 4400
+Wire Wire Line
+	6050 4300 6200 4300
+Wire Wire Line
+	6200 4300 6200 3900
+Wire Wire Line
+	6200 3900 6350 3900
+Connection ~ 6050 4300
+Wire Wire Line
+	7100 3900 6950 3900
+Wire Wire Line
+	4350 4300 4150 4300
+Wire Wire Line
+	4150 4300 4150 3650
+Wire Wire Line
+	4350 4150 4300 4150
+Wire Wire Line
+	4300 4150 4300 3650
+Wire Wire Line
+	4950 3700 4450 3700
+Wire Wire Line
+	4450 3700 4450 3650
+Wire Wire Line
+	5450 2700 5250 2700
+Wire Wire Line
+	4950 2700 4300 2700
+NoConn ~ 5100 3700
+NoConn ~ 5550 3700
+$Comp
+L debug-header DBG1
+U 1 1 56A3CC65
+P 6000 3350
+F 0 "DBG1" H 5650 3100 60  0000 C CNN
+F 1 "debug-header" H 6450 3100 60  0000 C CNN
+F 2 "footprints:debug" H 5350 3200 60  0000 C CNN
+F 3 "" H 6000 3350 60  0000 C CNN
+	1    6000 3350
+	-1   0    0    1
+$EndComp
+Wire Wire Line
+	5250 3700 5250 3350
+Wire Wire Line
+	5250 3350 5900 3350
+Wire Wire Line
+	5900 3350 5900 3200
+Wire Wire Line
+	5400 3700 5400 3400
+Wire Wire Line
+	5400 3400 6000 3400
+Wire Wire Line
+	6000 3400 6000 3200
+Text Label 5200 5300 3    60   ~ 0
+C2CK
+Text Label 5350 5300 3    60   ~ 0
+C2D
+Text Label 6100 3200 3    60   ~ 0
+C2CK
+Text Label 6200 3200 3    60   ~ 0
+C2D
 $EndSCHEMATC

Commit message: routed hot damn
Parts:
- removed DBG1: debug-header, footprints:debug, symbol debug-header
- added C2CK1, C2D1, RX1, TX1: debug-pin, footprints:debug, symbol debug-pin
- SW1: footprint footprints:MJTP1230 -> footprints:u2f-button
Connections:
- net labels added: RX, TX
- wire segments 45 -> 49
Changed lines of the file:
@@
 F 0 "SW1" H 6800 4010 50  0000 C CNN
 F 1 "SW_PUSH" H 6650 3820 50  0000 C CNN
-F 2 "footprints:MJTP1230" H 6650 3900 50  0001 C CNN
+F 2 "footprints:u2f-button" H 6650 3900 50  0001 C CNN
 F 3 "" H 6650 3900 50  0000 C CNN
 	1    6650 3900
@@
 	7100 3900 6950 3900
 Wire Wire Line
-	4350 4300 4150 4300
-Wire Wire Line
-	4150 4300 4150 3650
-Wire Wire Line
 	4350 4150 4300 4150
-Wire Wire Line
-	4300 4150 4300 3650
-Wire Wire Line
-	4950 3700 4450 3700
-Wire Wire Line
-	4450 3700 4450 3650
 Wire Wire Line
 	5450 2700 5250 2700
@@
 NoConn ~ 5100 3700
 NoConn ~ 5550 3700
-$Comp
-L debug-header DBG1
-U 1 1 56A3CC65
-P 6000 3350
-F 0 "DBG1" H 5650 3100 60  0000 C CNN
-F 1 "debug-header" H 6450 3100 60  0000 C CNN
-F 2 "footprints:debug" H 5350 3200 60  0000 C CNN
-F 3 "" H 6000 3350 60  0000 C CNN
-	1    6000 3350
-	-1   0    0    1
-$EndComp
 Wire Wire Line
-	5250 3700 5250 3350
+	5250 3700 5250 3300
 Wire Wire Line
-	5250 3350 5900 3350
+	5250 3300 5900 3300
 Wire Wire Line
-	5900 3350 5900 3200
+	5900 3300 5900 3200
 Wire Wire Line
 	5400 3700 5400 3400
@@
 Text Label 6200 3200 3    60   ~ 0
 C2D
+Wire Wire Line
+	4450 3650 4450 3900
+Wire Wire Line
+	4300 4150 4300 3900
+Wire Wire Line
+	4300 3900 4450 3900
+Wire Wire Line
+	4950 3700 4150 3700
+Wire Wire Line
+	4150 3700 4150 3650
+Wire Wire Line
+	4350 4300 4250 4300
+Wire Wire Line
+	4250 4300 4250 3800
+Wire Wire Line
+	4250 3800 4300 3800
+Wire Wire Line
+	4300 3800 4300 3650
+$Comp
+L debug-pin TX1
+U 1 1 56A3F7EB
+P 5700 3350
+F 0 "TX1" V 5500 2850 60  0000 C CNN
+F 1 "debug-pin" H 5800 3100 60  0001 C CNN
+F 2 "footprints:debug" H 5700 3350 60  0000 C CNN
+F 3 "" H 5700 3350 60  0000 C CNN
+	1    5700 3350
+	-1   0    0    1
+$EndComp
+$Comp
+L debug-pin RX1
+U 1 1 56A3F89E
+P 5800 3350
+F 0 "RX1" V 5600 2850 60  0000 C CNN
+F 1 "debug-pin" H 5900 3100 60  0001 C CNN
+F 2 "footprints:debug" H 5800 3350 60  0000 C CNN
+F 3 "" H 5800 3350 60  0000 C CNN
+	1    5800 3350
+	-1   0    0    1
+$EndComp
+$Comp
+L debug-pin C2CK1
+U 1 1 56A3F8D6
+P 5900 3350
+F 0 "C2CK1" V 5700 2800 60  0000 C CNN
+F 1 "debug-pin" H 6000 3100 60  0001 C CNN
+F 2 "footprints:debug" H 5900 3350 60  0000 C CNN
+F 3 "" H 5900 3350 60  0000 C CNN
+	1    5900 3350
+	-1   0    0    1
+$EndComp
+$Comp
+L debug-pin C2D1
+U 1 1 56A3F90D
+P 6000 3350
+F 0 "C2D1" V 5800 2800 60  0000 C CNN
+F 1 "debug-pin" H 6100 3100 60  0001 C CNN
+F 2 "footprints:debug" H 6000 3350 60  0000 C CNN
+F 3 "" H 6000 3350 60  0000 C CNN
+	1    6000 3350
+	-1   0    0    1
+$EndComp
+Text Label 5750 3300 0    60   ~ 0
+TX
+Text Label 5550 3400 0    60   ~ 0
+RX
 $EndSCHEMATC

Commit message: corrected pcb mistakes
Parts:
- removed C1: 0.1uF, Capacitors_SMD:C_0402, symbol C
- removed C2: 4.7uF, Capacitors_SMD:C_0603, symbol C
Connections:
- net +5V: now also A1.8 (VCC)
- net GND: now also E1.21 (GND), SW1.1; no longer SW1.2
- net HD+: now also E1.4 (D+), Z1.5 (C4); no longer E1.5 (D-), Z1.4 (C3)
- net HD-: now also E1.5 (D-), Z1.4 (C3); no longer E1.4 (D+), Z1.5 (C4)
- net at A1.5 (SDA): now also E1.2 (P0.0); no longer E1.13 (P1.1/SDA)
- net at A1.6 (SCL): now also E1.1 (P0.1); no longer E1.11 (P1.2/SCL)
- net at RGB1.1 (R): now also E1.14 (P1.0); no longer E1.1 (P0.1)
- net at E1.16 (P0.6): now also RGB1.3 (B)
- net at E1.19 (P0.3): now also E1.20 (P0.2), SW1.2
- net at RGB1.2 (G): now also E1.15 (P0.7); no longer E1.2 (P0.0)
- net +3.3V: no longer names the net of E1.6 (VDD)
- net +3.3V: no longer A1.8 (VCC)
- no-connect marks 8 -> 9
Other:
- moved on the sheet: A1, R1, RGB1, SW1
Changed lines of the file:
@@
 U 1 1 56857441
 P 5200 4500
-F 0 "E1" H 4800 5100 60  0000 C CNN
-F 1 "EFM8UB1" H 4650 5200 60  0000 C CNN
+F 0 "E1" H 5850 5100 60  0000 C CNN
+F 1 "EFM8UB1" H 5900 5200 60  0000 C CNN
 F 2 "footprints:EFM8UB1" H 4700 5000 60  0001 C CNN
 F 3 "" H 4700 5000 60  0000 C CNN
@@
 	1    0    0    -1
 $EndComp
-NoConn ~ 7600 4650
 $Comp
 L ATECC508A-RESCUE-u2f-zero A1
 U 1 1 56857313
-P 7000 4700
-F 0 "A1" H 7300 5000 60  0000 C CNN
-F 1 "ATECC508A" H 6900 5000 60  0000 C CNN
-F 2 "footprints:UDFN-8Pad" H 6600 4950 60  0001 C CNN
-F 3 "" H 6600 4950 60  0000 C CNN
-	1    7000 4700
-	-1   0    0    1
-$EndComp
-NoConn ~ 7600 4750
+P 4750 2350
+F 0 "A1" H 5050 2650 60  0000 C CNN
+F 1 "ATECC508A" H 4650 2650 60  0000 C CNN
+F 2 "footprints:UDFN-8Pad" H 4350 2600 60  0001 C CNN
+F 3 "" H 4350 2600 60  0000 C CNN
+	1    4750 2350
+	-1   0    0    1
+$EndComp
 Text Label 4350 4450 2    60   ~ 0
 GND
-NoConn ~ 7600 4850
-NoConn ~ 6400 4750
-Text Label 7850 5050 0    60   ~ 0
-GND
-Text Label 6400 5150 0    60   ~ 0
-+3.3V
 Text Label 6050 4700 0    60   ~ 0
 GND
@@
 	0    1    1    0
 $EndComp
-$Comp
-L C C1
-U 1 1 56858041
-P 4400 5600
-F 0 "C1" H 4425 5700 50  0000 L CNN
-F 1 "0.1uF" H 4425 5500 50  0000 L CNN
-F 2 "Capacitors_SMD:C_0402" H 4438 5450 50  0001 C CNN
-F 3 "" H 4400 5600 50  0000 C CNN
-	1    4400 5600
-	0    1    1    0
-$EndComp
-$Comp
-L C C2
-U 1 1 5685809E
-P 4400 5950
-F 0 "C2" H 4425 6050 50  0000 L CNN
-F 1 "4.7uF" H 4425 5850 50  0000 L CNN
-F 2 "Capacitors_SMD:C_0603" H 4438 5800 50  0001 C CNN
-F 3 "" H 4400 5950 50  0000 C CNN
-	1    4400 5950
-	0    1    1    0
-$EndComp
-Text Label 4050 6100 3    60   ~ 0
-GND
-Text Label 4750 5450 2    60   ~ 0
-+3.3V
-Text Label 5450 2700 0    60   ~ 0
+Text Label 4200 2900 0    60   ~ 0
 +5V
 $Comp
@@
 Text Label 3450 3900 2    60   ~ 0
 GND
-Text Label 3750 4600 0    60   ~ 0
+Text Label 3850 4750 0    60   ~ 0
 HD-
-Text Label 3950 4750 2    60   ~ 0
+Text Label 4050 4600 2    60   ~ 0
 HD+
-Text Label 7100 3900 0    60   ~ 0
-GND
 $Comp
 L R R1
 U 1 1 56857B9B
-P 5100 2700
-F 0 "R1" V 5180 2700 50  0000 C CNN
-F 1 "100" V 5100 2700 50  0000 C CNN
-F 2 "Resistors_SMD:R_0603" V 5030 2700 50  0001 C CNN
-F 3 "" H 5100 2700 50  0000 C CNN
-	1    5100 2700
-	0    1    1    0
+P 7750 4600
+F 0 "R1" V 7830 4600 50  0000 C CNN
+F 1 "100" V 7750 4600 50  0000 C CNN
+F 2 "Resistors_SMD:R_0603" V 7680 4600 50  0001 C CNN
+F 3 "" H 7750 4600 50  0000 C CNN
+	1    7750 4600
+	-1   0    0    1
 $EndComp
 NoConn ~ 5050 5300
@@
 Text Notes 3350 4900 0    60   ~ 0
 Host USB data
-Text Notes 6500 4350 0    60   ~ 0
+Text Notes 7450 3600 0    60   ~ 0
 Secure element for EC
 $Comp
 L CA_RGB-RESCUE-u2f-zero RGB1
 U 1 1 5686DEFD
-P 4500 3200
-F 0 "RGB1" H 4750 3350 60  0000 C CNN
-F 1 "CA_RGB" H 4400 3350 60  0000 C CNN
-F 2 "footprints:LED-0606" H 5300 3250 60  0001 C CNN
-F 3 "" H 4500 3250 60  0000 C CNN
-	1    4500 3200
-	0    1    -1   0
+P 7000 4450
+F 0 "RGB1" H 7250 4600 60  0000 C CNN
+F 1 "CA_RGB" H 6900 4600 60  0000 C CNN
+F 2 "footprints:LED-0606" H 7800 4500 60  0001 C CNN
+F 3 "" H 7000 4500 60  0000 C CNN
+	1    7000 4450
+	1    0    0    1
 $EndComp
 $Comp
@@
 	-1   0    0    1
 $EndComp
-Wire Wire Line
-	6050 4850 6300 4850
-Wire Wire Line
-	6300 4850 6300 4650
-Wire Wire Line
-	6300 4650 6400 4650
-Wire Wire Line
-	6400 4550 6050 4550
-Wire Wire Line
-	6400 4850 6400 5150
-Wire Wire Line
-	7600 4550 7850 4550
-Wire Wire Line
-	7850 4550 7850 5050
-Wire Wire Line
-	4900 5300 4900 6150
-Wire Wire Line
-	4900 5950 5200 5950
-Wire Wire Line
-	4900 5600 5200 5600
-Connection ~ 4900 5950
-Wire Wire Line
-	5500 5950 5750 5950
-Wire Wire Line
-	5750 5950 5750 5600
-Connection ~ 5750 5600
-Connection ~ 4900 5600
-Wire Wire Line
-	4750 5300 4750 5950
-Wire Wire Line
-	4750 5600 4550 5600
-Connection ~ 4750 5600
-Wire Wire Line
-	4050 5600 4250 5600
-Wire Wire Line
-	4750 5950 4550 5950
-Wire Wire Line
-	4050 5600 4050 6100
-Wire Wire Line
-	4050 5950 4250 5950
-Connection ~ 4050 5950
-Wire Wire Line
-	5500 5600 5900 5600
-Wire Wire Line
-	6850 5850 6850 5650
-Wire Wire Line
-	6550 5650 6550 5850
 Text Label 6850 5650 0    60   ~ 0
 +5V
@@
 L SW_PUSH SW1
 U 1 1 5685E9F9
-P 6650 3900
-F 0 "SW1" H 6800 4010 50  0000 C CNN
-F 1 "SW_PUSH" H 6650 3820 50  0000 C CNN
-F 2 "footprints:u2f-button" H 6650 3900 50  0001 C CNN
-F 3 "" H 6650 3900 50  0000 C CNN
-	1    6650 3900
-	1    0    0    -1
-$EndComp
-Wire Wire Line
-	3300 4600 3300 4750
-Wire Wire Line
-	3300 4750 4350 4750
-Wire Wire Line
-	3600 4600 4350 4600
+P 4750 3250
+F 0 "SW1" H 4900 3360 50  0000 C CNN
+F 1 "SW_PUSH" H 4750 3170 50  0000 C CNN
+F 2 "footprints:u2f-button" H 4750 3250 50  0001 C CNN
+F 3 "" H 4750 3250 50  0000 C CNN
+	1    4750 3250
+	1    0    0    -1
+$EndComp
 NoConn ~ 3250 4000
-Wire Wire Line
-	3450 4000 3450 3900
-Wire Wire Line
-	3650 4000 3650 3900
-Wire Wire Line
-	6050 4250 6050 4400
-Wire Wire Line
-	6050 4300 6200 4300
-Wire Wire Line
-	6200 4300 6200 3900
-Wire Wire Line
-	6200 3900 6350 3900
-Connection ~ 6050 4300
-Wire Wire Line
-	7100 3900 6950 3900
-Wire Wire Line
-	4350 4150 4300 4150
-Wire Wire Line
-	5450 2700 5250 2700
-Wire Wire Line
-	4950 2700 4300 2700
-NoConn ~ 5100 3700
-NoConn ~ 5550 3700
-Wire Wire Line
-	5250 3700 5250 3300
-Wire Wire Line
-	5250 3300 5900 3300
-Wire Wire Line
-	5900 3300 5900 3200
-Wire Wire Line
-	5400 3700 5400 3400
-Wire Wire Line
-	5400 3400 6000 3400
-Wire Wire Line
-	6000 3400 6000 3200
 Text Label 5200 5300 3    60   ~ 0
 C2CK
@@
 Text Label 6200 3200 3    60   ~ 0
 C2D
-Wire Wire Line
-	4450 3650 4450 3900
-Wire Wire Line
-	4300 4150 4300 3900
-Wire Wire Line
-	4300 3900 4450 3900
-Wire Wire Line
-	4950 3700 4150 3700
-Wire Wire Line
-	4150 3700 4150 3650
-Wire Wire Line
-	4350 4300 4250 4300
-Wire Wire Line
-	4250 4300 4250 3800
-Wire Wire Line
-	4250 3800 4300 3800
-Wire Wire Line
-	4300 3800 4300 3650
 $Comp
 L debug-pin TX1
@@
 F 0 "TX1" V 5500 2850 60  0000 C CNN
 F 1 "debug-pin" H 5800 3100 60  0001 C CNN
-F 2 "footprints:debug" H 5700 3350 60  0000 C CNN
+F 2 "footprints:debug" H 5700 3350 60  0001 C CNN
 F 3 "" H 5700 3350 60  0000 C CNN
 	1    5700 3350
@@
 F 0 "RX1" V 5600 2850 60  0000 C CNN
 F 1 "debug-pin" H 5900 3100 60  0001 C CNN
-F 2 "footprints:debug" H 5800 3350 60  0000 C CNN
+F 2 "footprints:debug" H 5800 3350 60  0001 C CNN
 F 3 "" H 5800 3350 60  0000 C CNN
 	1    5800 3350
@@
 F 0 "C2CK1" V 5700 2800 60  0000 C CNN
 F 1 "debug-pin" H 6000 3100 60  0001 C CNN
-F 2 "footprints:debug" H 5900 3350 60  0000 C CNN
+F 2 "footprints:debug" H 5900 3350 60  0001 C CNN
 F 3 "" H 5900 3350 60  0000 C CNN
 	1    5900 3350
@@
 F 0 "C2D1" V 5800 2800 60  0000 C CNN
 F 1 "debug-pin" H 6100 3100 60  0001 C CNN
-F 2 "footprints:debug" H 6000 3350 60  0000 C CNN
+F 2 "footprints:debug" H 5950 3500 60  0001 C CNN
 F 3 "" H 6000 3350 60  0000 C CNN
 	1    6000 3350
@@
 Text Label 5550 3400 0    60   ~ 0
 RX
+NoConn ~ 4750 5300
+NoConn ~ 4150 2400
+Text Label 5500 2200 0    60   ~ 0
+GND
+NoConn ~ 5350 2500
+NoConn ~ 5350 2400
+NoConn ~ 5350 2300
+Text Label 4450 3250 2    60   ~ 0
+GND
+Wire Wire Line
+	4900 5300 4900 6150
+Wire Wire Line
+	4900 5950 5200 5950
+Wire Wire Line
+	4900 5600 5200 5600
+Connection ~ 4900 5950
+Wire Wire Line
+	5500 5950 5750 5950
+Wire Wire Line
+	5750 5950 5750 5600
+Connection ~ 5750 5600
+Connection ~ 4900 5600
+Wire Wire Line
+	5500 5600 5900 5600
+Wire Wire Line
+	6850 5850 6850 5650
+Wire Wire Line
+	6550 5650 6550 5850
+Wire Wire Line
+	3300 4600 3300 4750
+Wire Wire Line
+	3450 4000 3450 3900
+Wire Wire Line
+	3650 4000 3650 3900
+Wire Wire Line
+	5250 3700 5250 3300
+Wire Wire Line
+	5250 3300 5900 3300
+Wire Wire Line
+	5900 3300 5900 3200
+Wire Wire Line
+	5400 3700 5400 3400
+Wire Wire Line
+	5400 3400 6000 3400
+Wire Wire Line
+	6000 3400 6000 3200
+Wire Wire Line
+	4150 2500 4100 2500
+Wire Wire Line
+	4100 2500 4100 2900
+Wire Wire Line
+	4100 2900 4200 2900
+Wire Wire Line
+	4150 2300 4050 2300
+Wire Wire Line
+	4050 2300 4050 4150
+Wire Wire Line
+	4050 4150 4350 4150
+Wire Wire Line
+	4150 2200 4000 2200
+Wire Wire Line
+	4000 2200 4000 4300
+Wire Wire Line
+	4000 4300 4350 4300
+Wire Wire Line
+	5350 2200 5500 2200
+Wire Wire Line
+	5100 3250 5100 3700
+Wire Wire Line
+	5100 3250 5050 3250
+Wire Wire Line
+	4950 3700 4950 3500
+Wire Wire Line
+	4950 3500 5100 3500
+Connection ~ 5100 3500
+Wire Wire Line
+	5550 3700 6350 3700
+Wire Wire Line
+	6350 3700 6350 4100
+Wire Wire Line
+	6350 4100 6550 4100
+Wire Wire Line
+	6050 4250 6550 4250
+Wire Wire Line
+	6550 4400 6050 4400
+Wire Wire Line
+	7500 4250 7750 4250
+Wire Wire Line
+	7750 4250 7750 4450
+Wire Wire Line
+	7750 4750 7750 4950
+Text Label 7750 4950 0    60   ~ 0
++5V
+Wire Wire Line
+	3300 4750 4350 4750
+Wire Wire Line
+	3600 4600 4350 4600
+NoConn ~ 6050 4550
+NoConn ~ 6050 4850
+Text Label 4850 3700 2    60   ~ 0
+GND
 $EndSCHEMATC
